Commit message: [UPD] fix position and rotations

File: open_manipulator_x_description/urdf/open_manipulator_x.urdf.xacro (robot description, xacro)
@@ -6,22 +6,22 @@
   <link name="omx1_platform_link">
     <visual>
-      <origin xyz="0 0 0" rpy="0 0 0"/>
-      <geometry>
-        <mesh filename="package://open_manipulator_x_description/meshes/omx1_link_base.stl" scale="0.001 0.001 0.001"/>
-      </geometry>
-      <material name="grey"/>
-    </visual>
-    <collision>
-      <origin xyz="0 0 0" rpy="0 0 0"/>
-      <geometry>
-        <mesh filename="package://open_manipulator_x_description/meshes/omx1_link_base.stl" scale="0.001 0.001 0.001"/>
-      </geometry>
-    </collision>
-    <inertial>
-      <origin xyz="0 0 0" />
-      <mass value="0.2" />
-      <inertia ixx="1.0-05" ixy="0.0" ixz="1.0-05"
-               iyy="1.0-05" iyz="0.0"
-               izz="1.0-05" />
+      <origin xyz="0 0 0" rpy="0 0 ${M_PI/2}"/>
+      <geometry>
+        <mesh filename="file://$(find open_manipulator_x_description)/meshes/omx1_link_base.stl" scale="0.001 0.001 0.001"/>
+      </geometry>
+      <material name="grey"/>
+    </visual>
+    <collision>
+      <origin xyz="0 0 0" rpy="0 0 ${M_PI/2}"/>
+      <geometry>
+        <mesh filename="file://$(find open_manipulator_x_description)/meshes/omx1_link_base.stl" scale="0.001 0.001 0.001"/>
+      </geometry>
+    </collision>
+    <inertial>
+      <origin xyz="0 0 0" rpy="0 0 ${M_PI/2}"/>
+      <mass value="0.2" />
+      <inertia ixx="1.0" ixy="0.0" ixz="1.0"
+               iyy="1.0" iyz="0.0"
+               izz="1.0" />
     </inertial>
   </link>
@@ -30,28 +30,27 @@
     <parent link="omx1_platform_link"/>
     <child link="omx1_base_link"/>
-    <origin xyz="0.0 0.0 0.0" rpy="0 0 0"/>
+    <origin xyz="-0.0105 -0.0135 0.006" rpy="0 0 0"/>
   </joint>
   <!-- Link 1: Base -->
   <link name="omx1_base_link">
     <visual>
-      <origin xyz="0 0 0" rpy="0 0 0"/>
-      <geometry>
-        <mesh filename="package://open_manipulator_x_description/meshes/omx1_link1.stl" scale="0.001 0.001 0.001"/>
-      </geometry>
-      <material name="grey"/>
-    </visual>
-    <collision>
-      <origin xyz="0 0 0" rpy="0 0 0"/>
-      <geometry>
-        <mesh filename="package://open_manipulator_x_description/meshes/omx1_link1.stl" scale="0.001 0.001 0.001"/>
-      </geometry>
-    </collision>
-    <inertial>
-      <origin xyz="0 0 0" />
-      <mass value="0.2" />
-      <inertia ixx="1.0-05" ixy="0.0" ixz="1.0-05"
-               iyy="1.0-05" iyz="0.0"
-               izz="1.0-05" />
-    </inertial>
+      <origin xyz="0 0 0" rpy="0 0 ${M_PI/2}"/>
+      <geometry>
+        <mesh filename="file://$(find open_manipulator_x_description)/meshes/omx1_link1.stl" scale="0.001 0.001 0.001"/>
+      </geometry>
+      <material name="grey"/>
+    </visual>
+    <collision>
+      <origin xyz="0 0 0" rpy="0 0 ${M_PI/2}"/>
+      <geometry>
+        <mesh filename="file://$(find open_manipulator_x_description)/meshes/omx1_link1.stl" scale="0.001 0.001 0.001"/>
+      </geometry>
+    </collision>
+    <inertial>
+      <origin xyz="0 0 0" rpy="0 0 ${M_PI/2}"/>
+      <mass value="0.2" />
+      <inertia ixx="1.0" ixy="0.0" ixz="1.0"
+               iyy="1.0" iyz="0.0"
+               izz="1.0" />
     </inertial>
   </link>
@@ -60,29 +59,29 @@
     <parent link="omx1_base_link"/>
     <child link="omx1_shoulder_link"/>
-    <origin xyz="0.0 0.0 0.0" rpy="0 0 0"/>
+    <origin xyz="0.0 0.0 0.0465" rpy="0 0 0"/>
     <axis xyz="0 0 1"/>
-    <limit velocity="4.8" effort="1" lower="-2.82743338823" upper="2.82743338823" />
+    <limit velocity="4.8" effort="1" lower="${-M_PI}" upper="${M_PI}" />
   </joint>
   <!--  Link 2: Shoulder -->
   <link name="omx1_shoulder_link">
     <visual>
-      <origin xyz="0 0 0.0" rpy="0 0 0"/>
-      <geometry>
-        <mesh filename="package://open_manipulator_x_description/meshes/omx1_link2.stl" scale="0.001 0.001 0.001"/>
-      </geometry>
-      <material name="grey"/>
-    </visual>
-    <collision>
-      <origin xyz="0 0 0.0" rpy="0 0 0"/>
-      <geometry>
-        <mesh filename="package://open_manipulator_x_description/meshes/omx1_link2.stl" scale="0.001 0.001 0.001"/>
-      </geometry>
-    </collision>
-    <inertial>
-      <origin xyz="0 0 0" />
-      <mass value="0.2" />
-      <inertia ixx="1.0-05" ixy="0.0" ixz="1.0-05"
-               iyy="1.0-05" iyz="0.0"
-               izz="1.0-05" />
+      <origin xyz="0 0 0.0" rpy="0 0 ${M_PI/2}"/>
+      <geometry>
+        <mesh filename="file://$(find open_manipulator_x_description)/meshes/omx1_link2.stl" scale="0.001 0.001 0.001"/>
+      </geometry>
+      <material name="grey"/>
+    </visual>
+    <collision>
+      <origin xyz="0 0 0.0" rpy="0 0 ${M_PI/2}"/>
+      <geometry>
+        <mesh filename="file://$(find open_manipulator_x_description)/meshes/omx1_link2.stl" scale="0.001 0.001 0.001"/>
+      </geometry>
+    </collision>
+    <inertial>
+      <origin xyz="0 0 0.0" rpy="0 0 ${M_PI/2}"/>
+      <mass value="0.2" />
+      <inertia ixx="1.0" ixy="0.0" ixz="1.0"
+               iyy="1.0" iyz="0.0"
+               izz="1.0" />
     </inertial>
   </link>
@@ -91,29 +90,29 @@
     <parent link="omx1_shoulder_link"/>
     <child link="omx1_upper_link"/>
-    <origin xyz="0.0 0.0 0.0" rpy="0 0 0"/>
+    <origin xyz="0.0 0.0 0.05095" rpy="0 0 0"/>
     <axis xyz="0 1 0"/>
-    <limit velocity="4.8" effort="1" lower="-1.79070781255" upper="1.57079632679" />
+    <limit velocity="4.8" effort="1" lower="${-M_PI/2}" upper="${M_PI/2}" />
   </joint>
   <!--  Link 3: Upper Arm -->
   <link name="omx1_upper_link">
     <visual>
-      <origin xyz="0 0 0" rpy="0 0 0"/>
-      <geometry>
-        <mesh filename="package://open_manipulator_x_description/meshes/omx1_link3.stl" scale="0.001 0.001 0.001"/>
-      </geometry>
-      <material name="grey"/>
-    </visual>
-    <collision>
-      <origin xyz="0 0 0" rpy="0 0 0"/>
-      <geometry>
-        <mesh filename="package://open_manipulator_x_description/meshes/omx1_link3.stl" scale="0.001 0.001 0.001"/>
-      </geometry>
-    </collision>
-    <inertial>
-      <origin xyz="0 0 0" />
-      <mass value="0.2" />
-      <inertia ixx="1.0-05" ixy="0.0" ixz="1.0-05"
-               iyy="1.0-05" iyz="0.0"
-               izz="1.0-05" />
+      <origin xyz="0 0 0" rpy="0 0 ${M_PI/2}"/>
+      <geometry>
+        <mesh filename="file://$(find open_manipulator_x_description)/meshes/omx1_link3.stl" scale="0.001 0.001 0.001"/>
+      </geometry>
+      <material name="grey"/>
+    </visual>
+    <collision>
+      <origin xyz="0 0 0" rpy="0 0 ${M_PI/2}"/>
+      <geometry>
+        <mesh filename="file://$(find open_manipulator_x_description)/meshes/omx1_link3.stl" scale="0.001 0.001 0.001"/>
+      </geometry>
+    </collision>
+    <inertial>
+      <origin xyz="0 0 0" rpy="0 0 ${M_PI/2}"/>
+      <mass value="0.2" />
+      <inertia ixx="1.0" ixy="0.0" ixz="1.0"
+               iyy="1.0" iyz="0.0"
+               izz="1.0" />
     </inertial>
   </link>
@@ -122,29 +121,29 @@
     <parent link="omx1_upper_link"/>
     <child link="omx1_lower_link"/>
-    <origin xyz="0.0 0 0.0" rpy="0 0 0"/>
+    <origin xyz="0.022 -0.0 0.128" rpy="0 0 0"/>
     <axis xyz="0 1 0"/>
-    <limit velocity="4.8" effort="1" lower="-0.94247779607" upper="1.38230076758" />
+    <limit velocity="4.8" effort="1" lower="${-M_PI/2}" upper="${M_PI/2}" />
   </joint>
   <!--  Link 4: Lower Arm -->
   <link name="omx1_lower_link">
     <visual>
-      <origin xyz="0 0 0" rpy="0 0 0"/>
-      <geometry>
-        <mesh filename="package://open_manipulator_x_description/meshes/omx1_link4.stl" scale="0.001 0.001 0.001"/>
-      </geometry>
-      <material name="grey"/>
-    </visual>
-    <collision>
-      <origin xyz="0 0 0" rpy="0 0 0"/>
-      <geometry>
-        <mesh filename="package://open_manipulator_x_description/meshes/omx1_link4.stl" scale="0.001 0.001 0.001"/>
-      </geometry>
-    </collision>
-    <inertial>
-      <origin xyz="0 0 0" />
-      <mass value="0.2" />
-      <inertia ixx="1.0-05" ixy="0.0" ixz="1.0-05"
-               iyy="1.0-05" iyz="0.0"
-               izz="1.0-05" />
+      <origin xyz="0 0 0" rpy="0 0 ${M_PI/2}"/>
+      <geometry>
+        <mesh filename="file://$(find open_manipulator_x_description)/meshes/omx1_link4.stl" scale="0.001 0.001 0.001"/>
+      </geometry>
+      <material name="grey"/>
+    </visual>
+    <collision>
+      <origin xyz="0 0 0" rpy="0 0 ${M_PI/2}"/>
+      <geometry>
+        <mesh filename="file://$(find open_manipulator_x_description)/meshes/omx1_link4.stl" scale="0.001 0.001 0.001"/>
+      </geometry>
+    </collision>
+    <inertial>
+      <origin xyz="0 0 0" rpy="0 0 ${M_PI/2}"/>
+      <mass value="0.2" />
+      <inertia ixx="1.0" ixy="0.0" ixz="1.0"
+               iyy="1.0" iyz="0.0"
+               izz="1.0" />
     </inertial>
   </link>
@@ -153,29 +152,29 @@
     <parent link="omx1_lower_link"/>
     <child link="omx1_forearm_roll_link"/>
-    <origin xyz="0.0 0.0 0.0" rpy="0 0 0"/>
-    <axis xyz="0 1 0"/>
-    <limit velocity="4.8" effort="1" lower="-1.79070781255" upper="2.04203522483" />
+    <origin xyz="0.0835 0.0 0.0" rpy="0 0 0"/>
+    <axis xyz="1 0 0"/>
+    <limit velocity="4.8" effort="1" lower="${-M_PI}" upper="${M_PI}" />
   </joint>
   <!--  Link 5: Forearm Upper -->
   <link name="omx1_forearm_roll_link">
     <visual>
-      <origin xyz="0 0 0" rpy="0 0 0"/>
-      <geometry>
-        <mesh filename="package://open_manipulator_x_description/meshes/omx1_link5.stl" scale="0.001 0.001 0.001"/>
-      </geometry>
-      <material name="grey"/>
-    </visual>
-    <collision>
-      <origin xyz="0 0 0" rpy="0 0 0"/>
-      <geometry>
-        <mesh filename="package://open_manipulator_x_description/meshes/omx1_link5.stl" scale="0.001 0.001 0.001"/>
-      </geometry>
-    </collision>
-    <inertial>
-      <origin xyz="0 0 0" />
-      <mass value="0.2" />
-      <inertia ixx="1.0-05" ixy="0.0" ixz="1.0-05"
-               iyy="1.0-05" iyz="0.0"
-               izz="1.0-05" />
+      <origin xyz="0 0 0" rpy="0 0 ${M_PI/2}"/>
+      <geometry>
+        <mesh filename="file://$(find open_manipulator_x_description)/meshes/omx1_link5.stl" scale="0.001 0.001 0.001"/>
+      </geometry>
+      <material name="grey"/>
+    </visual>
+    <collision>
+      <origin xyz="0 0 0" rpy="0 0 ${M_PI/2}"/>
+      <geometry>
+        <mesh filename="file://$(find open_manipulator_x_description)/meshes/omx1_link5.stl" scale="0.001 0.001 0.001"/>
+      </geometry>
+    </collision>
+    <inertial>
+      <origin xyz="0 0 0" rpy="0 0 ${M_PI/2}"/>
+      <mass value="0.2" />
+      <inertia ixx="1.0" ixy="0.0" ixz="1.0"
+               iyy="1.0" iyz="0.0"
+               izz="1.0" />
     </inertial>
   </link>
@@ -184,58 +183,60 @@
     <parent link="omx1_forearm_roll_link"/>
     <child link="omx1_forearm_tilt_link"/>
-    <origin xyz="0.0 0 0.0" rpy="0 0 0"/>
+    <origin xyz="0.0405 0.0 0.0" rpy="0 0 0"/>
     <axis xyz="0 1 0"/>
-    <limit velocity="4.8" effort="1" lower="-0.94247779607" upper="1.38230076758" />
+    <limit velocity="4.8" effort="1" lower="${-M_PI/2}" upper="${M_PI/2}" />
   </joint>
   <!--  Link 6: Forearm Lower -->
   <link name="omx1_forearm_tilt_link">
     <visual>
-      <origin xyz="0 0 0" rpy="0 0 0"/>
-      <geometry>
-        <mesh filename="package://open_manipulator_x_description/meshes/omx1_link6.stl" scale="0.001 0.001 0.001"/>
-      </geometry>
-      <material name="grey"/>
-    </visual>
-    <collision>
-      <origin xyz="0 0 0" rpy="0 0 0"/>
-      <geometry>
-        <mesh filename="package://open_manipulator_x_description/meshes/omx1_link6.stl" scale="0.001 0.001 0.001"/>
-      </geometry>
-    </collision>
-    <inertial>
-      <origin xyz="0 0 0" />
-      <mass value="0.2" />
-      <inertia ixx="1.0-05" ixy="0.0" ixz="1.0-05"
-               iyy="1.0-05" iyz="0.0"
-               izz="1.0-05" />
+      <origin xyz="0 0 0" rpy="0 0 ${M_PI/2}"/>
+      <geometry>
+        <mesh filename="file://$(find open_manipulator_x_description)/meshes/omx1_link6.stl" scale="0.001 0.001 0.001"/>
+      </geometry>
+      <material name="grey"/>
+    </visual>
+    <collision>
+      <origin xyz="0 0 0" rpy="0 0 ${M_PI/2}"/>
+      <geometry>
+        <mesh filename="file://$(find open_manipulator_x_description)/meshes/omx1_link6.stl" scale="0.001 0.001 0.001"/>
+      </geometry>
+    </collision>
+    <inertial>
+      <origin xyz="0 0 0" rpy="0 0 ${M_PI/2}"/>
+      <mass value="0.2" />
+      <inertia ixx="1.0" ixy="0.0" ixz="1.0"
+               iyy="1.0" iyz="0.0"
+               izz="1.0" />
     </inertial>
   </link>
   <!--  Joint 7: Wrist (Gripper Base) -->
-  <joint name="omx1_wrist_joint" type="fixed">
+  <joint name="omx1_wrist_joint" type="revolute">
     <parent link="omx1_forearm_tilt_link"/>
     <child link="omx1_wrist_link"/>
-    <origin xyz="0.0 0 0.0" rpy="0 0 0"/>
+    <origin xyz="0.064 0 0.0" rpy="0 0 0"/>
+    <axis xyz="1 0 0"/>
+    <limit velocity="4.8" effort="1" lower="${-M_PI}" upper="${M_PI}" />
   </joint>
   <!--  Link 7: Wrist (Gripper Base) -->
   <link name="omx1_wrist_link">
     <visual>
-      <origin xyz="0 0 0" rpy="0 0 0"/>
-      <geometry>
-        <mesh filename="package://open_manipulator_x_description/meshes/omx1_link7_gripper_base.stl" scale="0.001 0.001 0.001"/>
-      </geometry>
-      <material name="grey"/>
-    </visual>
-    <collision>
-      <origin xyz="0 0 0" rpy="0 0 0"/>
-      <geometry>
-        <mesh filename="package://open_manipulator_x_description/meshes/omx1_link7_gripper_base.stl" scale="0.001 0.001 0.001"/>
-      </geometry>
-    </collision>
-    <inertial>
-      <origin xyz="0 0 0" />
-      <mass value="0.2" />
-      <inertia ixx="1.0-05" ixy="0.0" ixz="1.0-05"
-               iyy="1.0-05" iyz="0.0"
-               izz="1.0-05" />
+      <origin xyz="0 0 0" rpy="0 0 ${M_PI/2}"/>
+      <geometry>
+        <mesh filename="file://$(find open_manipulator_x_description)/meshes/omx1_link7_gripper_base.stl" scale="0.001 0.001 0.001"/>
+      </geometry>
+      <material name="grey"/>
+    </visual>
+    <collision>
+      <origin xyz="0 0 0" rpy="0 0 ${M_PI/2}"/>
+      <geometry>
+        <mesh filename="file://$(find open_manipulator_x_description)/meshes/omx1_link7_gripper_base.stl" scale="0.001 0.001 0.001"/>
+      </geometry>
+    </collision>
+    <inertial>
+      <origin xyz="0 0 0" rpy="0 0 ${M_PI/2}"/>
+      <mass value="0.2" />
+      <inertia ixx="1.0" ixy="0.0" ixz="1.0"
+               iyy="1.0" iyz="0.0"
+               izz="1.0" />
     </inertial>
   </link>
@@ -244,27 +245,27 @@
     <parent link="omx1_wrist_link"/>
     <child link="omx1_gripper_link"/>
-    <origin xyz="0.0 0.0 0.0" rpy="0 0 0"/>
+    <origin xyz="0.05 0.0 0.0" rpy="0 0 0"/>
   </joint>
   <!--  Link 8: Gripper -->
   <link name="omx1_gripper_link">
     <visual>
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