Commit message: [UPD] upd links name

File: open_manipulator_x_description/urdf/open_manipulator_x.gazebo.xacro (robot description, xacro)
@@ -17,20 +17,36 @@
   <!-- World -->
   <gazebo reference="world"/>
-  <!-- Link1 -->
-  <RefLink ref="link1"/>
-  <!-- Link2 -->
-  <RefLink ref="link2"/>
-  <!-- Link3 -->
-  <RefLink ref="link3"/>
-  <!-- Link4 -->
-  <RefLink ref="link4"/>
-  <!-- Link5 -->
-  <RefLink ref="link5"/>
-  <!-- gripper_link -->
-  <RefLink ref="gripper_link"/>
-  <!-- gripper_link_sub -->
-  <RefLink ref="gripper_link_sub"/>
-  <!-- end effector link -->
-  <gazebo reference="end_effector_link">
+  <!-- Link 0: Platform -->
+  <RefLink ref="omx1_platform_link"/>
+  <!-- Link 1: Base -->
+  <RefLink ref="omx1_base_link"/>
+  <!-- Link 2: Shoulder -->
+  <RefLink ref="omx1_shoulder_link"/>
+  <!-- Link 3: Upper Arm -->
+  <RefLink ref="omx1_upper_link"/>
+  <!-- Link 4: Lower Arm -->
+  <RefLink ref="omx1_lower_link"/>
+  <!-- Link 5: Forearm Upper -->
+  <RefLink ref="omx1_forearm_roll_link"/>
+  <!-- Link 6: Forearm Lower -->
+  <RefLink ref="omx1_forearm_tilt_link"/>
+  <!-- Link 7: Wrist (Gripper Base) -->
+  <RefLink ref="omx1_wrist_link"/>
+  <!-- Link 8: Gripper -->
+  <RefLink ref="omx1_gripper_link"/>
+  <!-- Link 9: Gripper left sub -->
+  <RefLink ref="omx1_gripper_l_sub_link"/>
+  <!-- Link 10: Gripper right sub -->
+  <RefLink ref="omx1_gripper_r_sub_link"/>
+  <!-- Link 11: Gripper Finger Left -->
+  <RefLink ref="omx1_gripper_l_finger_link"/>
+  <!-- Link 12: Gripper Finger Right -->
+  <RefLink ref="omx1_gripper_r_finger_link"/>
+  <!-- Link 13: Gripper Tip Left -->
+  <RefLink ref="omx1_gripper_l_tip_link"/>
+  <!-- Link 14: Gripper Tip Right -->
+  <RefLink ref="omx1_gripper_r_tip_link"/>
+  <!-- Link 15: End Effector -->
+  <gazebo reference="omx1_end_effector_link">
     <material>Gazebo/Red</material>
   </gazebo>

File: open_manipulator_x_description/urdf/open_manipulator_x.transmission.xacro (robot description, xacro)
@@ -4,11 +4,11 @@
        xmlns:xacro="http://ros.org/wiki/xacro">
   <!-- Transmission macro -->
-  <xacro:macro name="SimpleTransmissionPosition" params="joint n">
-    <transmission name="tran${n}">
+  <xacro:macro name="SimpleTransmissionPosition" params="name">
+    <transmission name="${name}_tran">
       <type>transmission_interface/SimpleTransmission</type>
-      <joint name="${joint}">
+      <joint name="${name}_joint">
         <hardwareInterface>hardware_interface/PositionJointInterface</hardwareInterface>
       </joint>
-      <actuator name="motor${n}">
+      <actuator name="${name}_act">
         <mechanicalReduction>1</mechanicalReduction>
       </actuator>
@@ -16,26 +16,30 @@
   </xacro:macro>
   <!-- Transmission macro -->
-  <xacro:macro name="SimpleTransmissionEffort" params="joint n">
-    <transmission name="tran${n}">
+  <xacro:macro name="SimpleTransmissionEffort" params="name">
+    <transmission name="${name}_tran">
       <type>transmission_interface/SimpleTransmission</type>
-      <joint name="${joint}">
+      <joint name="${name}_joint">
         <hardwareInterface>hardware_interface/EffortJointInterface</hardwareInterface>
       </joint>
-      <actuator name="motor${n}">
+      <actuator name="${name}_act">
         <mechanicalReduction>1</mechanicalReduction>
       </actuator>
     </transmission>
   </xacro:macro>
-  <!-- Transmission 1 -->
-  <xacro:SimpleTransmissionPosition n="1" joint="joint1" />
-  <!-- Transmission 2 -->
-  <xacro:SimpleTransmissionPosition n="2" joint="joint2" />
-  <!-- Transmission 3 -->
-  <xacro:SimpleTransmissionPosition n="3" joint="joint3" />
-  <!-- Transmission 4 -->
-  <xacro:SimpleTransmissionPosition n="4" joint="joint4" />
-  <!-- Transmission 5 -->
-  <xacro:SimpleTransmissionEffort n="5" joint="gripper" />
-  <!-- Transmission 6 -->
-  <xacro:SimpleTransmissionEffort n="6" joint="gripper_sub" />
+  <!-- Transmission 1: Shoulder -->
+  <xacro:SimpleTransmissionPosition name="omx1_shoulder_link" />
+  <!-- Transmission 2: Upper Arm -->
+  <xacro:SimpleTransmissionPosition name="omx1_upper_link" />
+  <!-- Transmission 3: Lower Arm -->
+  <xacro:SimpleTransmissionPosition name="omx1_lower_link" />
+  <!-- Transmission 4: Forearm Upper -->
+  <xacro:SimpleTransmissionPosition name="omx1_forearm_roll_link" />
+  <!-- Transmission 5: Forearm Lower -->
+  <xacro:SimpleTransmissionPosition name="omx1_forearm_tilt_link" />
+  <!-- Transmission 6: Wrist (Gripper Base) -->
+  <xacro:SimpleTransmissionPosition name="omx1_wrist_link" />
+  <!-- Transmission 7: Gripper Finger Left -->
+  <xacro:SimpleTransmissionEffort name="omx1_gripper_l_finger_link" />
+  <!-- Transmission 8: Gripper Finger Right -->
+  <xacro:SimpleTransmissionEffort name="omx1_gripper_r_finger_link" />
 </robot>

Commit message: [FIX] rename with link number for order (temp)

File: open_manipulator_x_description/urdf/open_manipulator_x.gazebo.xacro (robot description, xacro)
@@ -22,15 +22,15 @@
   <RefLink ref="omx1_base_link"/>
   <!-- Link 2: Shoulder -->
-  <RefLink ref="omx1_shoulder_link"/>
+  <RefLink ref="omx1_arm1_link"/>
   <!-- Link 3: Upper Arm -->
-  <RefLink ref="omx1_upper_link"/>
+  <RefLink ref="omx1_arm2_link"/>
   <!-- Link 4: Lower Arm -->
-  <RefLink ref="omx1_lower_link"/>
+  <RefLink ref="omx1_arm3_link"/>
   <!-- Link 5: Forearm Upper -->
-  <RefLink ref="omx1_forearm_roll_link"/>
+  <RefLink ref="omx1_arm4_link"/>
   <!-- Link 6: Forearm Lower -->
-  <RefLink ref="omx1_forearm_tilt_link"/>
+  <RefLink ref="omx1_arm5_link"/>
   <!-- Link 7: Wrist (Gripper Base) -->
-  <RefLink ref="omx1_wrist_link"/>
+  <RefLink ref="omx1_arm6_link"/>
   <!-- Link 8: Gripper -->
   <RefLink ref="omx1_gripper_link"/>

File: open_manipulator_x_description/urdf/open_manipulator_x.transmission.xacro (robot description, xacro)
@@ -28,18 +28,18 @@
   </xacro:macro>
   <!-- Transmission 1: Shoulder -->
-  <xacro:SimpleTransmissionPosition name="omx1_shoulder_link" />
+  <xacro:SimpleTransmissionPosition name="omx1_arm1" />
   <!-- Transmission 2: Upper Arm -->
-  <xacro:SimpleTransmissionPosition name="omx1_upper_link" />
+  <xacro:SimpleTransmissionPosition name="omx1_arm2" />
   <!-- Transmission 3: Lower Arm -->
-  <xacro:SimpleTransmissionPosition name="omx1_lower_link" />
+  <xacro:SimpleTransmissionPosition name="omx1_arm3" />
   <!-- Transmission 4: Forearm Upper -->
-  <xacro:SimpleTransmissionPosition name="omx1_forearm_roll_link" />
+  <xacro:SimpleTransmissionPosition name="omx1_arm4" />
   <!-- Transmission 5: Forearm Lower -->
-  <xacro:SimpleTransmissionPosition name="omx1_forearm_tilt_link" />
+  <xacro:SimpleTransmissionPosition name="omx1_arm5" />
   <!-- Transmission 6: Wrist (Gripper Base) -->
-  <xacro:SimpleTransmissionPosition name="omx1_wrist_link" />
+  <xacro:SimpleTransmissionPosition name="omx1_arm6" />
   <!-- Transmission 7: Gripper Finger Left -->
-  <xacro:SimpleTransmissionEffort name="omx1_gripper_l_finger_link" />
+  <xacro:SimpleTransmissionEffort name="omx1_gripper_l_finger" />
   <!-- Transmission 8: Gripper Finger Right -->
-  <xacro:SimpleTransmissionEffort name="omx1_gripper_r_finger_link" />
+  <xacro:SimpleTransmissionEffort name="omx1_gripper_r_finger" />
 </robot>

File: open_manipulator_x_description/urdf/open_manipulator_x.urdf.xacro (robot description, xacro)
@@ -58,7 +58,7 @@
   </link>
   <!-- Joint 2: Shoulder -->
-  <joint name="omx1_shoulder_joint" type="revolute">
+  <joint name="omx1_arm1_joint" type="revolute">
     <parent link="omx1_base_link"/>
-    <child link="omx1_shoulder_link"/>
+    <child link="omx1_arm1_link"/>
     <origin xyz="0.0 0.0 0.0465" rpy="0 0 0"/>
     <axis xyz="0 0 1"/>
@@ -66,5 +66,5 @@
   </joint>
   <!--  Link 2: Shoulder -->
-  <link name="omx1_shoulder_link">
+  <link name="omx1_arm1_link">
     <visual>
       <origin xyz="0 0 0.0" rpy="0 0 ${M_PI/2}"/>
@@ -89,7 +89,7 @@
   </link>
   <!--  Joint 3: Upper Arm -->
-  <joint name="omx1_upper_joint" type="revolute">
-    <parent link="omx1_shoulder_link"/>
-    <child link="omx1_upper_link"/>
+  <joint name="omx1_arm2_joint" type="revolute">
+    <parent link="omx1_arm1_link"/>
+    <child link="omx1_arm2_link"/>
     <origin xyz="0.0 0.0 0.05095" rpy="0 0 0"/>
     <axis xyz="0 1 0"/>
@@ -97,5 +97,5 @@
   </joint>
   <!--  Link 3: Upper Arm -->
-  <link name="omx1_upper_link">
+  <link name="omx1_arm2_link">
     <visual>
       <origin xyz="0 0 0" rpy="0 0 ${M_PI/2}"/>
@@ -120,7 +120,7 @@
   </link>
   <!--  Joint 4: Lower Arm -->
-  <joint name="omx1_lower_joint" type="revolute">
-    <parent link="omx1_upper_link"/>
-    <child link="omx1_lower_link"/>
+  <joint name="omx1_arm3_joint" type="revolute">
+    <parent link="omx1_arm2_link"/>
+    <child link="omx1_arm3_link"/>
     <origin xyz="0.022 -0.0 0.128" rpy="0 0 0"/>
     <axis xyz="0 1 0"/>
@@ -128,5 +128,5 @@
   </joint>
   <!--  Link 4: Lower Arm -->
-  <link name="omx1_lower_link">
+  <link name="omx1_arm3_link">
     <visual>
       <origin xyz="0 0 0" rpy="0 0 ${M_PI/2}"/>
@@ -151,7 +151,7 @@
   </link>
   <!--  Joint 5: Forearm Upper -->
-  <joint name="omx1_forearm_upper_joint" type="revolute">
-    <parent link="omx1_lower_link"/>
-    <child link="omx1_forearm_roll_link"/>
+  <joint name="omx1_arm4_joint" type="revolute">
+    <parent link="omx1_arm3_link"/>
+    <child link="omx1_arm4_link"/>
     <origin xyz="0.0835 0.0 0.0" rpy="0 0 0"/>
     <axis xyz="1 0 0"/>
@@ -159,5 +159,5 @@
   </joint>
   <!--  Link 5: Forearm Upper -->
-  <link name="omx1_forearm_roll_link">
+  <link name="omx1_arm4_link">
     <visual>
       <origin xyz="0 0 0" rpy="0 0 ${M_PI/2}"/>
@@ -182,7 +182,7 @@
   </link>
   <!--  Joint 6: Forearm Lower -->
-  <joint name="omx1_forearm_lower_link" type="revolute">
-    <parent link="omx1_forearm_roll_link"/>
-    <child link="omx1_forearm_tilt_link"/>
+  <joint name="omx1_arm5_joint" type="revolute">
+    <parent link="omx1_arm4_link"/>
+    <child link="omx1_arm5_link"/>
     <origin xyz="0.0405 0.0 0.0" rpy="0 0 0"/>
     <axis xyz="0 1 0"/>
@@ -190,5 +190,5 @@
   </joint>
   <!--  Link 6: Forearm Lower -->
-  <link name="omx1_forearm_tilt_link">
+  <link name="omx1_arm5_link">
     <visual>
       <origin xyz="0 0 0" rpy="0 0 ${M_PI/2}"/>
@@ -213,7 +213,7 @@
   </link>
   <!--  Joint 7: Wrist (Gripper Base) -->
-  <joint name="omx1_wrist_joint" type="revolute">
-    <parent link="omx1_forearm_tilt_link"/>
-    <child link="omx1_wrist_link"/>
+  <joint name="omx1_arm6_joint" type="revolute">
+    <parent link="omx1_arm5_link"/>
+    <child link="omx1_arm6_link"/>
     <origin xyz="0.064 0 0.0" rpy="0 0 0"/>
     <axis xyz="1 0 0"/>
@@ -221,5 +221,5 @@
   </joint>
   <!--  Link 7: Wrist (Gripper Base) -->
-  <link name="omx1_wrist_link">
+  <link name="omx1_arm6_link">
     <visual>
       <origin xyz="0 0 0" rpy="0 0 ${M_PI/2}"/>
@@ -245,5 +245,5 @@
   <!--  Joint 8: Gripper -->
   <joint name="omx1_gripper_joint" type="fixed">
-    <parent link="omx1_wrist_link"/>
+    <parent link="omx1_arm6_link"/>
     <child link="omx1_gripper_link"/>
     <origin xyz="0.05 0.0 0.0" rpy="0 0 0"/>
@@ -454,5 +454,5 @@
   <joint name="end_effector_joint" type="fixed">
     <origin xyz="${0.0935+0.0375/2} 0.0 0.0" rpy="0 0 0"/>
-    <parent link="omx1_wrist_link"/>
+    <parent link="omx1_arm6_link"/>
     <child link="omx1_end_effector_link"/>
   </joint>
